File: diseño/kicad/esquematico_esp32/esquematico_esp32.kicad_sch (KiCad schematic)
At the start: 0 parts

Commit message: design v1.0
Parts:
- added BT1: 12V, symbol Device:Battery
- added J1, J10, J2, J3, J4, J5, J6, J7, J8, J9: Conn_01x02_Pin, symbol Connector:Conn_01x02_Pin
- added JP1: Jumper_2_Open, symbol Jumper:Jumper_2_Open
- added R1: R, symbol Device:R
- added U1: ~, symbol componentes aguas:esp32_heltec
- added U10, U5, U6: TIP110, TO-220_STM, symbol 2025-05-21_07-05-57:TIP110
- added U2: ~, symbol componentes aguas:sensor_presion
- added U3: ~, symbol componentes aguas:74218A
- added U4: ULN2003A, symbol Transistor_Array:ULN2003A
- added U7, U8, U9: 2N6517, TO-92-3L_5P33X5P2_ONS, symbol 2025-05-21_07-22-19:2N6517
Connections:
- new net: J7.1 (Pin_1), U4.14 (O3)
- new net: U10.1, U9.1 (E)
- new net: J10.1 (Pin_1), U10.2, U9.3 (C)
- new net: U5.1, U8.1 (E)
- new net: J1.1 (Pin_1), U5.2, U8.3 (C)
- new net: J9.1 (Pin_1), R1.1, U1. (GND)
- new net: JP1.1 (A), U1. (GND)
- new net: J6.1 (Pin_1), U4.13 (O4)
- new net: U6.1, U7.1 (E)
- new net: J2.1 (Pin_1), U6.2, U7.3 (C)
- new net: J5.1 (Pin_1), U4.12 (O5)
- new net: J4.1 (Pin_1), U4.11 (O6)
- new net: J8.1 (Pin_1), U4.15 (O2)
- new net: J3.1 (Pin_1), U4.10 (O7)
- new net 12V: BT1.1 (+), J2.2 (Pin_2)
- new net 3V3: U1. (GND), U2. (Vcc), U3. (RESN)
- new net 5V: J1.2 (Pin_2), J10.2 (Pin_2), J3.2 (Pin_2), J4.2 (Pin_2), J5.2 (Pin_2), J6.2 (Pin_2), J7.2 (Pin_2), J8.2 (Pin_2), J9.2 (Pin_2), JP1.2 (B)
- new net BOMBA 1: U1. (GND), U4.7 (I7)
- new net BOMBA 2: U1. (GND), U4.6 (I6)
- new net BOMBA 3: U1. (GND), U4.5 (I5)
- new net BOMBA 4: U1. (GND), U4.4 (I4)
- new net GND: BT1.2 (-), R1.2, U1. (GND), U10.3, U2. (Vcc), U3. (RESN), U4.8 (GND), U5.3, U6.3
- new net LED 1: U1. (GND), U8.2 (B)
- new net LED 2: U1. (GND), U7.2 (B)
- new net LED 3: U1. (GND), U9.2 (B)
- new net SCL: U1. (GND), U2. (Vcc), U3. (RESN)
- new net SDA: U1. (GND), U2. (Vcc), U3. (RESN)
- new net Sensor: U1. (GND)
- new net VALVULA 1: U1. (GND), U4.2 (I2)
- new net VALVULA 2: U1. (GND), U4.3 (I3)
- no-connect marks 0 -> 24
Other:
- note added: "B1"
- note added: "B2"
- note added: "B3"
- note added: "B4"
- note added: "Led1"
- note added: "Led2"
- note added: "Led3"
- note added: "Sensor"
- note added: "V1"
- note added: "V2"

Commit message: v1.1
Connections:
- net SCL: no longer U2. (Vcc)
- net SDA: no longer U2. (Vcc)
- new net: U1. (GND), U2. (Vcc) (x2)
- no-connect marks 24 -> 22
Changed lines of the file:
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@@
-	)
-	(junction
-		(at 83.82 27.94)
-		(diameter 0)
-		(color 0 0 0 0)
 	)
 	(junction
@@
 	)
 	(junction
-		(at 82.55 35.56)
+		(at 39.37 53.34)
+		(diameter 0)
+		(color 0 0 0 0)
+	)
+	(junction
+		(at 74.93 91.44)
+		(diameter 0)
+		(color 0 0 0 0)
+	)
+	(junction
+		(at 85.09 33.02)
+		(diameter 0)
+		(color 0 0 0 0)
+	)
+	(junction
+		(at 40.64 50.8)
 		(diameter 0)
 		(color 0 0 0 0)
@@
 	)
 	(junction
-		(at 39.37 53.34)
-		(diameter 0)
-		(color 0 0 0 0)
-	)
-	(junction
-		(at 74.93 91.44)
-		(diameter 0)
-		(color 0 0 0 0)
-	)
-	(junction
-		(at 85.09 33.02)
-		(diameter 0)
-		(color 0 0 0 0)
-	)
-	(junction
-		(at 40.64 50.8)
-		(diameter 0)
-		(color 0 0 0 0)
-	)
-	(junction
 		(at 248.92 71.12)
 		(diameter 0)
@@
 	)
 	(no_connect
-		(at 62.23 40.64)
-	)
-	(no_connect
 		(at 62.23 45.72)
 	)
 	(no_connect
-		(at 62.23 41.91)
-	)
-	(no_connect
 		(at 119.38 39.37)
 	)
@@
 	(wire
 		(pts
+			(xy 83.82 40.64) (xy 62.23 40.64)
+		)
+		(stroke
+			(width 0)
+			(type default)
+		)
+	)
+	(wire
+		(pts
 			(xy 22.86 48.26) (xy 22.86 45.72)
 		)
@@
 	(wire
 		(pts
+			(xy 82.55 46.99) (xy 82.55 41.91)
+		)
+		(stroke
+			(width 0)
+			(type default)
+		)
+	)
+	(wire
+		(pts
 			(xy 39.37 25.4) (xy 39.37 53.34)
 		)
@@
 	(wire
 		(pts
-			(xy 82.55 35.56) (xy 82.55 46.99)
-		)
-		(stroke
-			(width 0)
-			(type default)
-		)
-	)
-	(wire
-		(pts
 			(xy 54.61 62.23) (xy 27.94 62.23)
 		)
@@
 	(wire
 		(pts
+			(xy 81.28 25.4) (xy 81.28 46.99)
+		)
+		(stroke
+			(width 0)
+			(type default)
+		)
+	)
+	(wire
+		(pts
 			(xy 142.24 92.71) (xy 142.24 96.52)
 		)
@@
 	(wire
 		(pts
-			(xy 95.25 27.94) (xy 83.82 27.94)
-		)
-		(stroke
-			(width 0)
-			(type default)
-		)
-	)
-	(wire
-		(pts
 			(xy 30.48 40.64) (xy 30.48 45.72)
 		)
@@
 	(wire
 		(pts
-			(xy 83.82 27.94) (xy 83.82 46.99)
-		)
-		(stroke
-			(width 0)
-			(type default)
-		)
-	)
-	(wire
-		(pts
 			(xy 74.93 38.1) (xy 62.23 38.1)
 		)
@@
 	(wire
 		(pts
-			(xy 82.55 35.56) (xy 40.64 35.56)
+			(xy 40.64 35.56) (xy 96.52 35.56)
 		)
 		(stroke
@@
 	(wire
 		(pts
-			(xy 81.28 25.4) (xy 39.37 25.4)
+			(xy 39.37 25.4) (xy 81.28 25.4)
 		)
 		(stroke
@@
 	(wire
 		(pts
-			(xy 81.28 25.4) (xy 81.28 46.99)
-		)
-		(stroke
-			(width 0)
-			(type default)
-		)
-	)
-	(wire
-		(pts
 			(xy 93.98 44.45) (xy 93.98 25.4)
 		)
@@
 	(wire
 		(pts
+			(xy 83.82 46.99) (xy 83.82 40.64)
+		)
+		(stroke
+			(width 0)
+			(type default)
+		)
+	)
+	(wire
+		(pts
 			(xy 54.61 49.53) (xy 54.61 62.23)
 		)
@@
 	(wire
 		(pts
-			(xy 96.52 35.56) (xy 82.55 35.56)
-		)
-		(stroke
-			(width 0)
-			(type default)
-		)
-	)
-	(wire
-		(pts
 			(xy 43.18 49.53) (xy 43.18 50.8)
 		)
@@
 	(wire
 		(pts
+			(xy 81.28 25.4) (xy 93.98 25.4)
+		)
+		(stroke
+			(width 0)
+			(type default)
+		)
+	)
+	(wire
+		(pts
 			(xy 92.71 44.45) (xy 92.71 33.02)
 		)
@@
 	(wire
 		(pts
+			(xy 82.55 41.91) (xy 62.23 41.91)
+		)
+		(stroke
+			(width 0)
+			(type default)
+		)
+	)
+	(wire
+		(pts
 			(xy 27.94 40.64) (xy 30.48 40.64)
 		)
@@
 	(wire
 		(pts
-			(xy 83.82 27.94) (xy 43.18 27.94)
+			(xy 43.18 27.94) (xy 95.25 27.94)
 		)
 		(stroke
@@
 		)
 		(stroke
-			(width 0)
-			(type default)
-		)
-	)
-	(wire
-		(pts
-			(xy 93.98 25.4) (xy 81.28 25.4)
-		)
-		(stroke

Commit message: version final sin valvulas y bombas
Connections:
- new net: U1. (GND), U2. (Vcc) (x2)
Other:
- moved on the sheet: BT1, U4
Changed lines of the file:
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@@
 	)
 	(no_connect
-		(at 119.38 39.37)
+		(at 121.92 39.37)
 	)
 	(no_connect
@@
 	)
 	(no_connect
-		(at 119.38 44.45)
+		(at 121.92 44.45)
 	)
 	(no_connect
@@
 	)
 	(no_connect
-		(at 139.7 44.45)
+		(at 142.24 44.45)
 	)
 	(no_connect
@@
 	(wire
 		(pts
-			(xy 139.7 59.69) (xy 143.51 59.69)
+			(xy 142.24 59.69) (xy 143.51 59.69)
 		)
 		(stroke
@@
 	(wire
 		(pts
-			(xy 139.7 57.15) (xy 143.51 57.15)
+			(xy 142.24 57.15) (xy 143.51 57.15)
 		)
 		(stroke
@@
 	(wire
 		(pts
-			(xy 110.49 54.61) (xy 119.38 54.61)
-		)
-		(stroke
-			(width 0)
-			(type default)
-		)
-	)
-	(wire
-		(pts
-			(xy 107.95 49.53) (xy 119.38 49.53)
+			(xy 110.49 54.61) (xy 121.92 54.61)
+		)
+		(stroke
+			(width 0)
+			(type default)
+		)
+	)
+	(wire
+		(pts
+			(xy 107.95 49.53) (xy 121.92 49.53)
 		)
 		(stroke
@@
 	(wire
 		(pts
-			(xy 30.48 133.35) (xy 30.48 137.16)
+			(xy 26.67 102.87) (xy 26.67 106.68)
 		)
 		(stroke
@@
 	(wire
 		(pts
-			(xy 139.7 49.53) (xy 143.51 49.53)
+			(xy 142.24 49.53) (xy 143.51 49.53)
 		)
 		(stroke
@@
 	(wire
 		(pts
-			(xy 119.38 59.69) (xy 119.38 67.31)
-		)
-		(stroke
-			(width 0)
-			(type default)
-		)
-	)
-	(wire
-		(pts
 			(xy 27.94 38.1) (xy 31.75 38.1)
 		)
@@
 	(wire
 		(pts
-			(xy 139.7 52.07) (xy 143.51 52.07)
+			(xy 142.24 52.07) (xy 143.51 52.07)
 		)
 		(stroke
@@
 	(wire
 		(pts
-			(xy 121.92 95.25) (xy 121.92 67.31)
+			(xy 121.92 59.69) (xy 121.92 95.25)
 		)
 		(stroke
@@
 	(wire
 		(pts
+			(xy 132.08 64.77) (xy 129.54 64.77)
+		)
+		(stroke
+			(width 0)
+			(type default)
+		)
+	)
+	(wire
+		(pts
 			(xy 74.93 38.1) (xy 62.23 38.1)
 		)
@@
 	(wire
 		(pts
-			(xy 121.92 67.31) (xy 119.38 67.31)
-		)
-		(stroke
-			(width 0)
-			(type default)
-		)
-	)
-	(wire
-		(pts
 			(xy 27.94 30.48) (xy 35.56 30.48)
 		)
@@
 	(wire
 		(pts
-			(xy 139.7 54.61) (xy 143.51 54.61)
+			(xy 142.24 54.61) (xy 143.51 54.61)
 		)
 		(stroke
@@
 	(wire
 		(pts
-			(xy 106.68 46.99) (xy 119.38 46.99)
+			(xy 106.68 46.99) (xy 121.92 46.99)
 		)
 		(stroke
@@
 	(wire
 		(pts
-			(xy 30.48 147.32) (xy 30.48 148.59)
-		)
-		(stroke
-			(width 0)
-			(type default)
-		)
-	)
-	(wire
-		(pts
-			(xy 109.22 52.07) (xy 119.38 52.07)
+			(xy 26.67 116.84) (xy 26.67 118.11)
+		)
+		(stroke
+			(width 0)
+			(type default)
+		)
+	)
+	(wire
+		(pts
+			(xy 109.22 52.07) (xy 121.92 52.07)
 		)
 		(stroke
@@
 	(wire
 		(pts
-			(xy 139.7 46.99) (xy 143.51 46.99)
+			(xy 142.24 46.99) (xy 143.51 46.99)
 		)
 		(stroke
@@
 	(wire
 		(pts
-			(xy 114.3 57.15) (xy 119.38 57.15)
+			(xy 114.3 57.15) (xy 121.92 57.15)
 		)
 		(stroke
@@
 	(hierarchical_label "12V"
 		(shape input)
-		(at 30.48 133.35 90)
+		(at 26.67 102.87 90)
 		(effects
 			(font
@@
 	(symbol
 		(lib_id "Device:Battery")
-		(at 30.48 142.24 0)
+		(at 26.67 111.76 0)
 		(unit 1)
 		(exclude_from_sim no)
@@
 		(fields_autoplaced yes)
 		(property "Reference" "BT1"
-			(at 34.29 140.3984 0)
+			(at 30.48 109.9184 0)
 			(effects
 				(font
@@
 		)
 		(property "Value" "12V"
-			(at 34.29 142.9384 0)
+			(at 30.48 112.4584 0)
 			(effects
 				(font
@@
 		)
 		(property "Footprint" ""
-			(at 30.48 140.716 90)
+			(at 26.67 110.236 90)
 			(effects
 				(font
@@
 		)
 		(property "Datasheet" "~"
-			(at 30.48 140.716 90)
+			(at 26.67 110.236 90)
 			(effects
 				(font
@@
 		)
 		(property "Description" "Multiple-cell battery"
-			(at 30.48 142.24 0)
+			(at 26.67 111.76 0)
 			(effects
 				(font
@@
 	(symbol
 		(lib_id "power:GND")
-		(at 30.48 148.59 0)
+		(at 26.67 118.11 0)
 		(unit 1)
 		(exclude_from_sim no)
@@
 		(fields_autoplaced yes)
 		(property "Reference" "#PWR06"
-			(at 30.48 154.94 0)
+			(at 26.67 124.46 0)
 			(effects
 				(font
@@
 		)
 		(property "Value" "GND"
-			(at 30.48 153.67 0)
+			(at 26.67 123.19 0)
 			(effects
 				(font
@@
 		)
 		(property "Footprint" ""
-			(at 30.48 148.59 0)
+			(at 26.67 118.11 0)
 			(effects
 				(font
@@
 		)
 		(property "Datasheet" ""
-			(at 30.48 148.59 0)
+			(at 26.67 118.11 0)
 			(effects
 				(font
@@
 		)
 		(property "Description" "Power symbol creates a global label with name \"GND\" , ground"
-			(at 30.48 148.59 0)
+			(at 26.67 118.11 0)
 			(effects
 				(font
@@
 	(symbol
 		(lib_id "Transistor_Array:ULN2003A")
-		(at 129.54 49.53 0)
+		(at 132.08 49.53 0)
 		(mirror y)
 		(unit 1)
@@
 		(dnp no)
 		(property "Reference" "U4"
-			(at 129.54 31.75 0)
+			(at 132.08 31.75 0)
 			(effects
 				(font
@@
 		)
 		(property "Value" "ULN2003A"
-			(at 129.54 34.29 0)
+			(at 132.08 34.29 0)
 			(effects
 				(font
@@
 		)
 		(property "Footprint" ""
-			(at 128.27 63.5 0)
+			(at 130.81 63.5 0)
 			(effects
 				(font
@@
 		)
 		(property "Datasheet" "http://www.ti.com/lit/ds/symlink/uln2003a.pdf"
-			(at 127 54.61 0)
+			(at 129.54 54.61 0)
 			(effects
 				(font
@@
 		)
 		(property "Description" "High Voltage, High Current Darlington Transistor Arrays, SOIC16/SOIC16W/DIP16/TSSOP16"
-			(at 129.54 49.53 0)
-			(effects
-				(font
+			(at 132.08 49.53 0)
+			(effects
+				(font
